File: HARDWARE/iW-CORE-BOARD.kicad_pcb (KiCad board)
At the start: 2 copper layers, 115 x 72 mm, 0 parts

Commit message: Pre position of components
Parts:
- added BT1: 3V, BS-12-B-___002:BS-12-B-1A, B.Cu at (98.5, 72.0)
- added C1: 0.1uF, Capacitor_SMD:C_0603_1608Metric, B.Cu at (209.7, 111.7)
- added C10: 10pF, Capacitor_SMD:C_0603_1608Metric, B.Cu at (213.7, 109.2)
- added C11: 22pF, Capacitor_SMD:C_0603_1608Metric, B.Cu at (213.7, 106.7)
- added C12: 22pF, Capacitor_SMD:C_0603_1608Metric, B.Cu at (213.7, 104.2)
- added C13: 0.1uF, Capacitor_SMD:C_0603_1608Metric, B.Cu at (213.7, 101.6)
- added C14: 0.1uF, Capacitor_SMD:C_0603_1608Metric, B.Cu at (213.7, 99.1)
- added C15: 1uF, Capacitor_SMD:C_0603_1608Metric, B.Cu at (213.7, 96.6)
- added C16: 0.1uF, Capacitor_SMD:C_0603_1608Metric, B.Cu at (236.7, 74.0)
- added C17: 10uF, Capacitor_SMD:C_0603_1608Metric, B.Cu at (214.9, 156.7)
- added C18: 10uF, Capacitor_SMD:C_0603_1608Metric, B.Cu at (214.9, 154.2)
- added C19: 22uF, Capacitor_SMD:C_0603_1608Metric, B.Cu at (214.9, 151.7)
- added C2: 0.1uF, Capacitor_SMD:C_0603_1608Metric, B.Cu at (209.7, 109.2)
- added C20: 22uF, Capacitor_SMD:C_0603_1608Metric, B.Cu at (214.9, 149.2)
- added C21: 22uF, Capacitor_SMD:C_0603_1608Metric, B.Cu at (214.9, 146.7)
- added C22: 10uF, Capacitor_SMD:C_0603_1608Metric, B.Cu at (214.9, 144.2)
- added C23: 10uF, Capacitor_SMD:C_0603_1608Metric, B.Cu at (218.9, 156.7)
- added C3: 0.1uF, Capacitor_SMD:C_0603_1608Metric, B.Cu at (209.7, 106.7)
- added C32: 0.1uF, Capacitor_SMD:C_0603_1608Metric, B.Cu at (213.7, 94.1)
- added C33: 0.1uF, Capacitor_SMD:C_0603_1608Metric, B.Cu at (209.7, 74.0)
- added C34: 0.1uF, Capacitor_SMD:C_0603_1608Metric, B.Cu at (209.7, 71.5)
- added C36: 100nF, Capacitor_SMD:C_0603_1608Metric, B.Cu at (217.7, 111.7)
- added C37: 0.1uF, Capacitor_SMD:C_0603_1608Metric, B.Cu at (217.7, 109.2)
- added C38: 10uF, Capacitor_SMD:C_0805_2012Metric, B.Cu at (252.1, 120.2)
- added C39: 1uF, Capacitor_SMD:C_0603_1608Metric, B.Cu at (262.5, 87.1)
- added C4: 0.1uF, Capacitor_SMD:C_0603_1608Metric, B.Cu at (209.7, 104.2)
- added C40: 100nF, Capacitor_SMD:C_0603_1608Metric, B.Cu at (262.5, 84.6)
- added C41: 100nf, Capacitor_SMD:C_0603_1608Metric, B.Cu at (262.5, 82.1)
- added C42: 1uF, Capacitor_SMD:C_0603_1608Metric, B.Cu at (262.5, 79.6)
- added C43: 100nF, Capacitor_SMD:C_0603_1608Metric, B.Cu at (218.9, 154.2)
- added C44: 10uF, Capacitor_SMD:C_0603_1608Metric, B.Cu at (218.9, 151.7)
- added C45: 100nF, Capacitor_SMD:C_0603_1608Metric, B.Cu at (218.9, 149.2)
- added C46: 10uF, Capacitor_SMD:C_0603_1608Metric, B.Cu at (218.9, 146.7)
- added C47: 0.1uF, Capacitor_SMD:C_0603_1608Metric, B.Cu at (217.7, 106.7)
- added C48: 0.1uF, Capacitor_SMD:C_0603_1608Metric, B.Cu at (236.7, 71.5)
- added C49: 100nF, Capacitor_SMD:C_0603_1608Metric, B.Cu at (233.4, 127.5)
- added C5: 0.1uF, Capacitor_SMD:C_0603_1608Metric, B.Cu at (209.7, 101.6)
- added C50: 100nF, Capacitor_SMD:C_0603_1608Metric, B.Cu at (233.4, 125.0)
- added C6: 4.7uF, Capacitor_SMD:C_0603_1608Metric, B.Cu at (209.7, 99.1)
- added C7: 2.2uF, Capacitor_SMD:C_0603_1608Metric, B.Cu at (209.7, 96.6)
- added C8: 2.2uF, Capacitor_SMD:C_0603_1608Metric, B.Cu at (209.7, 94.1)
- added C9: 10pF, Capacitor_SMD:C_0603_1608Metric, B.Cu at (213.7, 111.7)
- added D1: LED, LED_SMD:LED_0603_1608Metric, B.Cu at (226.9, 148.3)
- added D10: LED, LED_SMD:LED_0603_1608Metric, B.Cu at (226.9, 145.7)
- added D11: LED, LED_SMD:LED_0603_1608Metric, B.Cu at (220.6, 86.7)
- added D12: LED, LED_SMD:LED_0603_1608Metric, B.Cu at (220.6, 84.1)
- added D13: LED, LED_SMD:LED_0603_1608Metric, B.Cu at (220.6, 81.5)
- added D3: BAT54C, Package_TO_SOT_SMD:SOT-23, B.Cu at (225.0, 81.0)
- added D4: LED, LED_SMD:LED_0603_1608Metric, B.Cu at (230.6, 74.0)
- added D7: ESD9B3.3ST5G, Diode_SMD:D_SOD-923, B.Cu at (255.3, 103.5)
- added FB1: 600R, Inductor_SMD:L_0603_1608Metric, B.Cu at (217.7, 104.2)
- added FB2: 600R, Inductor_SMD:L_0603_1608Metric, B.Cu at (233.4, 122.5)
- added FB3: 600R, Inductor_SMD:L_0603_1608Metric, B.Cu at (233.4, 120.0)
- added H1: MountingHole, MountingHole:MountingHole_2.5mm_Pad, F.Cu at (88.9, 64.0)
- added H2: MountingHole, MountingHole:MountingHole_2.5mm_Pad, F.Cu at (200.0, 64.0)
- added H3: MountingHole, MountingHole:MountingHole_2.5mm_Pad, F.Cu at (88.9, 136.0)
- added H4: MountingHole, MountingHole:MountingHole_2.5mm_Pad, F.Cu at (200.0, 136.0)
- added J1: Conn_01x40_MountingPin, Connector_FFC-FPC:TE_4-1734839-0_1x40-1MP_P0.5mm_Horizontal, F.Cu at (124.7, 104.4)
- added J2: Conn_01x06_MountingPin, Connector_FFC-FPC:TE_0-1734839-6_1x06-1MP_P0.5mm_Horizontal, F.Cu at (172.6, 105.1)
- added J3: 1746142-1, KiCad:17461421, B.Cu at (135.5, 137.4)
- added J4: Conn_02x09_Counter_Clockwise, Connector_IDC:IDC-Header_2x09_P2.54mm_Vertical_SMD, B.Cu at (99.7, 104.3)
- added J5: Conn_02x09_Counter_Clockwise, Connector_IDC:IDC-Header_2x09_P2.54mm_Vertical_SMD, B.Cu at (191.4, 103.5)
- added J6: Conn_02x05_Odd_Even, Connector_PinHeader_1.27mm:PinHeader_2x05_P1.27mm_Vertical_SMD, B.Cu at (191.4, 126.0)
- added J7: USB_C_Receptacle_USB2.0, Connector_USB:USB_C_Receptacle_G-Switch_GT-USB-7010ASV, B.Cu at (165.7, 135.9)
- added J8: Conn_02x05_Odd_Even, Connector_PinHeader_1.27mm:PinHeader_2x05_P1.27mm_Vertical_SMD, B.Cu at (179.9, 85.0)
- added J9: USB_C_Receptacle_USB2.0, Connector_USB:USB_C_Receptacle_G-Switch_GT-USB-7010ASV, B.Cu at (178.5, 136.0)
- added JP1: SolderJumper_2_Open, Jumper:SolderJumper-2_P1.3mm_Open_Pad1.0x1.5mm, B.Cu at (252.0, 127.0)
- added JP2: SolderJumper_2_Open, Jumper:SolderJumper-2_P1.3mm_Open_Pad1.0x1.5mm, B.Cu at (252.0, 123.4)
- added L1: 1uH, Inductor_SMD:L_0603_1608Metric, B.Cu at (218.9, 144.2)
- added L2: 10uH, Inductor_SMD:L_0805_2012Metric, B.Cu at (246.8, 119.7)
- added P1: ST-TF-003A, ST-TF-003A:SUNTECH_ST-TF-003A, B.Cu at (118.2, 69.2)
- added R1: 0R, Resistor_SMD:R_0603_1608Metric, B.Cu at (217.7, 101.6)
- added R11: 10k, Resistor_SMD:R_0603_1608Metric, B.Cu at (222.9, 154.2)
- added R12: 2R, Resistor_SMD:R_0603_1608Metric, B.Cu at (222.9, 151.7)
- added R2: 10k, Resistor_SMD:R_0603_1608Metric, B.Cu at (217.7, 99.1)
- added R28: 33R, Resistor_SMD:R_0603_1608Metric, B.Cu at (217.7, 96.6)
- added R29: 33R, Resistor_SMD:R_0603_1608Metric, B.Cu at (217.7, 94.1)
- added R3: 47k, Resistor_SMD:R_0603_1608Metric, B.Cu at (236.7, 69.0)
- added R30: 33R, Resistor_SMD:R_0603_1608Metric, B.Cu at (221.7, 111.7)
- added R31: 33R, Resistor_SMD:R_0603_1608Metric, B.Cu at (221.7, 109.2)
- added R32: 33R, Resistor_SMD:R_0603_1608Metric, B.Cu at (221.7, 106.7)
- added R33: 100k, Resistor_SMD:R_0603_1608Metric, B.Cu at (221.7, 104.2)
- added R34: 22R, Resistor_SMD:R_0603_1608Metric, B.Cu at (221.7, 101.6)
- added R35: 22R, Resistor_SMD:R_0603_1608Metric, B.Cu at (221.7, 99.1)
- added R36: 22R, Resistor_SMD:R_0603_1608Metric, B.Cu at (221.7, 96.6)
- added R37: 22R, Resistor_SMD:R_0603_1608Metric, B.Cu at (221.7, 94.1)
- added R38: 100R, Resistor_SMD:R_0603_1608Metric, B.Cu at (225.7, 111.7)
- added R39: 10k, Resistor_SMD:R_0603_1608Metric, B.Cu at (225.7, 109.2)
- added R4: 47k, Resistor_SMD:R_0603_1608Metric, B.Cu at (236.7, 66.5)
- added R40: 100R, Resistor_SMD:R_0603_1608Metric, B.Cu at (209.7, 69.0)
- added R41: 22R, Resistor_SMD:R_0603_1608Metric, B.Cu at (209.7, 66.5)
- added R42: 22R, Resistor_SMD:R_0603_1608Metric, B.Cu at (209.7, 64.0)
- added R44: 22R, Resistor_SMD:R_0603_1608Metric, B.Cu at (209.7, 61.5)
- added R45: 470R, Resistor_SMD:R_0603_1608Metric, B.Cu at (222.9, 149.2)
- added R46: 5k, Resistor_SMD:R_0603_1608Metric, B.Cu at (237.4, 127.5)
- added R47: 10R, Resistor_SMD:R_0603_1608Metric, B.Cu at (237.4, 125.0)
- added R48: 10k, Resistor_SMD:R_0603_1608Metric, B.Cu at (237.4, 122.5)
- added R49: 10k, Resistor_SMD:R_0603_1608Metric, B.Cu at (237.4, 120.0)
- added R5: 47k, Resistor_SMD:R_0603_1608Metric, B.Cu at (236.7, 64.0)
- added R50: 220R, Resistor_SMD:R_0603_1608Metric, B.Cu at (209.7, 59.0)
- added R51: 220R, Resistor_SMD:R_0603_1608Metric, B.Cu at (209.7, 56.4)
- added R52: 470R, Resistor_SMD:R_0603_1608Metric, B.Cu at (225.7, 106.7)
- added R53: 470R, Resistor_SMD:R_0603_1608Metric, B.Cu at (225.7, 104.2)
- added R54: 470R, Resistor_SMD:R_0603_1608Metric, B.Cu at (225.7, 101.6)
- added R6: 47k, Resistor_SMD:R_0603_1608Metric, B.Cu at (236.7, 61.5)
- added R7: 47k, Resistor_SMD:R_0603_1608Metric, B.Cu at (236.7, 59.0)
- added R8: 47k, Resistor_SMD:R_0603_1608Metric, B.Cu at (236.7, 56.4)
- added R9: 2R, Resistor_SMD:R_0603_1608Metric, B.Cu at (222.9, 156.7)
- added SW1: SW_Push, Button_Switch_SMD:SW_SPST_CK_RS282G05A3, B.Cu at (166.0, 89.1)
- added SW2: SW_Push, Button_Switch_SMD:SW_SPST_CK_RS282G05A3, B.Cu at (160.8, 89.1)
- added SW3: SW_Push, Button_Switch_SMD:SW_SPST_CK_RS282G05A3, B.Cu at (157.0, 121.5)
- added U1: STM32H750VBTx, Package_QFP:LQFP-100_14x14mm_P0.5mm, B.Cu at (157.5, 107.0)
- added U10: USBLC6-2SC6, Package_TO_SOT_SMD:SOT-23-6, B.Cu at (166.0, 126.5)
- added U11: USBLC6-2SC6, Package_TO_SOT_SMD:SOT-23-6, B.Cu at (179.0, 127.0)
- added U12: LT3465, Package_TO_SOT_SMD:TSOT-23-6, B.Cu at (242.0, 118.7)
- added U2: IP5306, IP5306:SOP8-P, B.Cu at (227.9, 153.8)
- added U3: STM32F072CBT6, Package_QFP:LQFP-48_7x7mm_P0.5mm, B.Cu at (174.5, 118.5)
- added U7: W25Q256JVS, Package_SON:WSON-8-1EP_8x6mm_P1.27mm_EP3.4x4.3mm, B.Cu at (174.8, 96.4)
- added U9: AMS1117-3.3, Package_TO_SOT_SMD:SOT-223-3_TabPin2, B.Cu at (151.0, 89.5)
- added Y1: 8MHz, Crystal:Crystal_SMD_Abracon_ABM3-2Pin_5.0x3.2mm, B.Cu at (239.0, 96.5)
- added Y2: 32.768KHz, Crystal:Crystal_SMD_3215-2Pin_3.2x1.5mm, B.Cu at (251.3, 102.8)
Other:
- board size 115 x 72 mm -> 118 x 80 mm
- copper layers 2 -> 4
