File: HARDWARE/_autosave-iW-CORE-BOARD.kicad_pcb (KiCad board)
At the start: 4 copper layers, 118 x 80 mm, 121 parts, among them J1 Conn_01x40_MountingPin, J2 Conn_01x06_MountingPin, J3 1746142-1, J4 Conn_02x09_Counter_Clockwise, J5 Conn_02x09_Counter_Clockwise, J6 Conn_02x05_Odd_Even, J7 USB_C_Receptacle_USB2.0, J8 Conn_02x05_Odd_Even, J9 USB_C_Receptacle_USB2.0, P1 ST-TF-003A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

Commit message: Placement
Parts:
- moved JP1 163.7 mm to (96.0, 77.5)
- moved C41 162.5 mm to (100.0, 86.5)
- moved JP2 161.6 mm to (96.0, 81.5)
- moved C38 158.3 mm to (99.8, 77.2)
- moved C39 156.5 mm to (106.0, 90.0), turned to 90 degrees
- moved C40 154.6 mm to (108.0, 90.0), turned to 90 degrees
- moved C42 153.1 mm to (109.5, 86.2), turned to 90 degrees
- moved L2 148.8 mm to (103.5, 79.5)
- moved R46 143.8 mm to (100.1, 84.5)
- moved U12 140.2 mm to (105.8, 85.6), turned to 90 degrees
- moved R47 140.1 mm to (102.8, 86.0), turned to 90 degrees
- moved FB3 139.9 mm to (99.5, 79.5)
- moved R48 128.9 mm to (110.5, 100.0), turned to -90 degrees
- moved FB2 127.8 mm to (109.8, 90.0), turned to 90 degrees
- moved C50 126.6 mm to (108.5, 104.0), turned to -90 degrees
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