File: HARDWARE/DISPLAY.kicad_sch (KiCad schematic)
At the start: 19 parts, among them J1 Conn_01x40_MountingPin, J2 Conn_01x06_MountingPin, U12 LT3465

Commit message: Pre position of components
Changed lines of the file:
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@@
 	)
 	(global_label "LTDC_HSYNC"
-		(shape output)
+		(shape input)
 		(at 147.32 105.41 180)
 		(fields_autoplaced yes)
@@
 	)
 	(global_label "LTDC_B4"
-		(shape output)
+		(shape input)
 		(at 147.32 87.63 180)
 		(fields_autoplaced yes)
@@
 	)
 	(global_label "LTDC_CLK"
-		(shape output)
+		(shape input)
 		(at 147.32 100.33 180)
 		(fields_autoplaced yes)
@@
 	)
 	(global_label "LTDC_R4"
-		(shape output)
+		(shape input)
 		(at 147.32 46.99 180)
 		(fields_autoplaced yes)
@@
 	)
 	(global_label "LTDC_G2"
-		(shape output)
+		(shape input)
 		(at 147.32 62.23 180)
 		(fields_autoplaced yes)
@@
 	)
 	(global_label "LTDC_G5"
-		(shape output)
+		(shape input)
 		(at 147.32 69.85 180)
 		(fields_autoplaced yes)
@@
 	)
 	(global_label "LTDC_R7"
-		(shape output)
+		(shape input)
 		(at 147.32 54.61 180)
 		(fields_autoplaced yes)
@@
 	)
 	(global_label "LTDC_G4"
-		(shape output)
+		(shape input)
 		(at 147.32 67.31 180)
 		(fields_autoplaced yes)
@@
 	)
 	(global_label "LTDC_G6"
-		(shape output)
+		(shape input)
 		(at 147.32 72.39 180)
 		(fields_autoplaced yes)
@@
 	)
 	(global_label "LTDC_G3"
-		(shape output)
+		(shape input)
 		(at 147.32 64.77 180)
 		(fields_autoplaced yes)
@@
 	)
 	(global_label "LTDC_B6"
-		(shape output)
+		(shape input)
 		(at 147.32 92.71 180)
 		(fields_autoplaced yes)
@@
 	)
 	(global_label "LTDC_R3"
-		(shape output)
+		(shape input)
 		(at 147.32 44.45 180)
 		(fields_autoplaced yes)
@@
 	)
 	(global_label "LTDC_B3"
-		(shape output)
+		(shape input)
 		(at 147.32 85.09 180)
 		(fields_autoplaced yes)
@@
 	)
 	(global_label "LTDC_VSYNC"
-		(shape output)
+		(shape input)
 		(at 147.32 107.95 180)
 		(fields_autoplaced yes)
@@
 	)
 	(global_label "LTDC_B7"
-		(shape output)
+		(shape input)
 		(at 147.32 95.25 180)
 		(fields_autoplaced yes)
@@
 	)
 	(global_label "LTDC_G7"
-		(shape output)
+		(shape input)
 		(at 147.32 74.93 180)
 		(fields_autoplaced yes)
@@
 	)
 	(global_label "LTDC_DE"
-		(shape output)
+		(shape input)
 		(at 147.32 110.49 180)
 		(fields_autoplaced yes)
@@
 	)
 	(global_label "LTDC_R5"
-		(shape output)
+		(shape input)
 		(at 147.32 49.53 180)
 		(fields_autoplaced yes)
@@
 	)
 	(global_label "LTDC_B5"
-		(shape output)
+		(shape input)
 		(at 147.32 90.17 180)
 		(fields_autoplaced yes)
@@
 	)
 	(global_label "LTDC_B2"
-		(shape output)
+		(shape input)
 		(at 147.32 82.55 180)
 		(fields_autoplaced yes)
@@
 	)
 	(global_label "LTDC_R6"
-		(shape output)
+		(shape input)
 		(at 147.32 52.07 180)
 		(fields_autoplaced yes)
@@
 	)
 	(global_label "LTDC_R2"
-		(shape output)
+		(shape input)
 		(at 147.32 41.91 180)
 		(fields_autoplaced yes)

Commit message: ada
Parts:
- L2: footprint Inductor_SMD:L_0805_2012Metric -> Inductor_SMD:L_1210_3225Metric
Changed lines of the file:
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@@
 			)
 		)
-		(property "Footprint" "Inductor_SMD:L_0805_2012Metric"
+		(property "Footprint" "Inductor_SMD:L_1210_3225Metric"
 			(at 70.866 47.244 0)
 			(effects
