File: HARDWARE/DISPLAY.kicad_sch (KiCad schematic)
At the start: 19 parts, among them J1 Conn_01x40_MountingPin, J2 Conn_01x06_MountingPin, U12 LT3465

Commit message: fix fpc
Parts:
- removed C50: 100nF, Capacitor_SMD:C_0603_1608Metric, symbol Device:C_Small
- removed JP1, JP2: SolderJumper_2_Open, Jumper:SolderJumper-2_P1.3mm_Open_Pad1.0x1.5mm, symbol Jumper:SolderJumper_2_Open
- removed R49: 10k, Resistor_SMD:R_0603_1608Metric, symbol Device:R_Small
Connections:
- net 3.3V is gone; now on net +3.3V: J2.1 (Pin_1)
- net +5V: now also C38.1, FB3.1
- net GND: now also J2.MP (MountPin)
- net +3V3 renamed +3.3V
- no-connect marks 0 -> 5
Other:
- moved on the sheet: C49, J1, J2, R48

Commit message: fix lcd
Parts:
- added R10, R13: 2.2k, Resistor_SMD:R_0603_1608Metric, symbol Device:R_Small
Connections:
- net +3.3V: now also R10.1, R13.1
- net I2C3_SCL: now also R10.2
- net I2C3_SDA: now also R13.2
