File: HARDWARE/JTAG.kicad_sch (KiCad schematic)
At the start: 16 parts, among them J8 Conn_02x05_Odd_Even, J9 USB_C_Receptacle_USB2.0, U11 USBLC6-2SC6, U3 STM32F072CBT6

Commit message: ada
Parts:
- removed R40: 100R, Resistor_SMD:R_0603_1608Metric, symbol Device:R_Small
Connections:
- net +5VBUS: no longer C33.1
- net +5V_USB_JLOB: now reaches J9.A4 (VBUS), J9.A9 (VBUS), J9.B4 (VBUS), J9.B9 (VBUS)
- net +5V_USB_JLOB: now also C33.1
