File: HARDWARE/JTAG.kicad_sch (KiCad schematic)
At the start: 13 parts, among them J8 Conn_02x05_Odd_Even, J9 USB_C_Receptacle_USB2.0, U11 USBLC6-2SC6, U3 STM32F072CBT6

Commit message: Pre position of components
Changed lines of the file:
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@@
 	)
 	(global_label "UART7_TX"
-		(shape bidirectional)
+		(shape input)
 		(at 165.1 87.63 0)
 		(fields_autoplaced yes)
@@
 		)
 		(property "Intersheetrefs" "${INTERSHEET_REFS}"
-			(at 178.2074 87.63 0)
+			(at 177.0961 87.63 0)
 			(effects
 				(font
@@
 	)
 	(global_label "SDMMC2_D2"
-		(shape output)
+		(shape input)
 		(at 165.1 69.85 0)
 		(fields_autoplaced yes)
@@
 	)
 	(global_label "SWDCLK_OB"
-		(shape output)
+		(shape input)
 		(at 242.57 119.38 0)
 		(fields_autoplaced yes)
@@
 	)
 	(global_label "SWDCLK"
-		(shape output)
+		(shape input)
 		(at 180.34 67.31 0)
 		(fields_autoplaced yes)
@@
 		)
 		(property "Intersheetrefs" "${INTERSHEET_REFS}"
-			(at 190.7448 67.31 0)
+			(at 190.8242 67.31 0)
 			(effects
 				(font
@@
 	)
 	(global_label "UART7_RX"
-		(shape bidirectional)
+		(shape output)
 		(at 165.1 85.09 0)
 		(fields_autoplaced yes)
@@
 		)
 		(property "Intersheetrefs" "${INTERSHEET_REFS}"
-			(at 178.5098 85.09 0)
+			(at 177.3985 85.09 0)
 			(effects
 				(font
@@
 	)
 	(global_label "NRST_OB"
-		(shape output)
+		(shape input)
 		(at 242.57 127 0)
 		(fields_autoplaced yes)

Commit message: Fix componentes possiton
Connections:
- net USB_OB_N: no longer J9.A7 (D-), J9.B7 (D-), U11.1 (I/O1)
- net USB_OB_P: no longer J9.A6 (D+), J9.B6 (D+), U11.3 (I/O2)
- new net USB_O_N: J9.A7 (D-), J9.B7 (D-), U11.1 (I/O1)
- new net USB_O_P: J9.A6 (D+), J9.B6 (D+), U11.3 (I/O2)
Changed lines of the file:
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@@
 		)
 	)
-	(label "USB_OB_N"
+	(label "USB_O_N"
 		(at 229.87 68.58 0)
 		(effects
@@
 		)
 	)
-	(label "USB_OB_P"
+	(label "USB_O_P"
 		(at 229.87 92.71 0)
 		(effects

Commit message: esa
Parts:
- added C35, C51, C52: 0.1uF, Capacitor_SMD:C_0603_1608Metric, symbol Device:C_Small
Connections:
- net +3.3V: now also C35.1, C51.1, C52.1
- net GND: now also C35.2, C51.2, C52.2
Other:
- moved on the sheet: C34

Commit message: fix fpc
Parts:
- removed J8: Conn_02x05_Odd_Even, Connector_PinHeader_1.27mm:PinHeader_2x05_P1.27mm_Vertical_SMD, symbol Connector_Generic:Conn_02x05_Odd_Even
- removed R40: 100R, Resistor_SMD:R_0603_1608Metric, symbol Device:R_Small
- removed R41, R42, R44: 22R, Resistor_SMD:R_0603_1608Metric, symbol Device:R_Small
Connections:
- net +5VBUS is gone; now on net +5V_COM: C33.1, U11.5 (VBUS)
- net +5V_COM: now reaches J9.A4 (VBUS), J9.A9 (VBUS), J9.B4 (VBUS), J9.B9 (VBUS)
- no-connect marks 6 -> 4
Other:
- note removed: "DEBUG & PROG"
