File: HARDWARE/POWER.kicad_sch (KiCad schematic)
At the start: 26 parts, among them J3 1746142-1, SW3 SW_Push, U2 IP5306, U9 AMS1117-3.3

Commit message: ada
Parts:
- added D2, D5: SS34, Diode_SMD:D_SMA, symbol Diode:SS34
- C17, C18, C22: footprint Capacitor_SMD:C_0603_1608Metric -> Capacitor_SMD:C_0805_2012Metric
Connections:
- net +5VBUS: no longer names the net of C18.1, R9.1, U2.1 (VIN)
- net +5VBUS: now also D2.1 (K), D5.1 (K)
- new net +5V_USBCOM: D2.2 (A)
- new net +5V_USB_JLOB: D5.2 (A)
